Commit message: fix: tune Nav2 footprint and low-speed limits

File: src/ylhb_base/urdf/ylhb.urdf.xacro (robot description, xacro)
@@ -3,10 +3,10 @@
   <!-- 1. 定义主要参考坐标系 (通常位于机器人底盘中心在地面的投影位置) -->
   <link name="base_footprint"/>
-  <!-- 2. 小车主体框架：建立 base_link（设位于轮间距中心，尺寸 30x30 cm） -->
+  <!-- 2. 小车主体框架：建立 base_link（实测长方体包络） -->
   <link name="base_link">
     <visual>
+      <origin xyz="0.0885 0 0.07175" rpy="0 0 0"/>
       <geometry>
-        <!-- 小车大致是个长宽 0.3x0.3m 的板，假设厚度为2cm -->
-        <box size="0.3 0.3 0.02"/>
+        <box size="0.465 0.470 0.3165"/>
       </geometry>
       <material name="gray">
@@ -14,11 +14,16 @@
       </material>
     </visual>
+    <collision>
+      <origin xyz="0.0885 0 0.07175" rpy="0 0 0"/>
+      <geometry>
+        <box size="0.465 0.470 0.3165"/>
+      </geometry>
+    </collision>
   </link>
-  <!-- 将 base_link 与 base_footprint 链接。假设当前车轮半径为 3cm(0.03m)
-       如果这里设为0，则代表轮距中心就在地板贴地上。 -->
+  <!-- 将 base_link 与 base_footprint 链接，保持底盘坐标系在轮间中心。 -->
   <joint name="footprint_to_base_joint" type="fixed">
     <parent link="base_footprint"/>
     <child link="base_link"/>
-    <origin xyz="0 0 0.03" rpy="0 0 0"/>
+    <origin xyz="0 0 0.0865" rpy="0 0 0"/>
   </joint>
   <!-- 3. 定义 IMU 的位置与物理属性 -->

Commit message: fix: calibrate ZLAC drive mapping and sensor frames

File: src/ylhb_base/urdf/ylhb.urdf.xacro (robot description, xacro)
@@ -57,5 +57,5 @@
     <child link="imu_link"/>
     <!-- 匹配 ROS 前左上标准坐标系 (X为前，Y为左，Z为上) -->
-    <origin xyz="0.280 0 0.107" rpy="0 0 0"/>
+    <origin xyz="-0.280 0 0.107" rpy="0 0 0"/>
   </joint>
   <joint name="base_to_laser_joint" type="fixed">
@@ -65,5 +65,5 @@
          这意味着雷达自身的 X轴 指向了小车的右侧 (-Y方向)。
          因此，雷达坐标系相对于小车主坐标系顺时针旋转了90度，即 Yaw = -1.5707963 -->
-    <origin xyz="0.090 0 0.1805" rpy="0 0 -1.5707963"/>
+    <origin xyz="-0.090 0 0.1805" rpy="0 0 -1.5707963"/>
   </joint>
 </robot>
